Commit message: updates

File: franka_robotiq/urdf/fr3_robotiq.urdf.xacro (robot description, xacro)
@@ -41,4 +41,5 @@
   <xacro:arg name="com_port" default='/dev/ttyUSB0' />
   <xacro:arg name="index" default='0' />
+  <xacro:arg name="ft_sensor" default="false" />
   <xacro:franka_robotiq arm_id="$(arg arm_id)"
                       joint_limits="${xacro.load_yaml('$(find franka_description)/robots/fr3/joint_limits.yaml')}"
@@ -59,4 +60,5 @@
                       connected_to= "base"
                       index="$(arg index)"
+                      ft_sensor="$(arg ft_sensor)"
                       xyz="$(arg xyz)"
                       rpy="$(arg rpy)"

File: franka_robotiq/urdf/franka_arm.ros2_control.xacro (robot description, xacro)
@@ -18,4 +18,5 @@
     <ros2_control name="${arm_prefix_modified}FrankaHardwareInterface" type="system">
         <hardware>
+          <param name="version">0.1.0</param>
           <param name="arm_id">${arm_id}</param>
           <param name="prefix">${arm_prefix}</param>

File: franka_robotiq/urdf/franka_robotiq.xacro (robot description, xacro)
@@ -13,4 +13,5 @@
                       ee_id:='franka_hand'
                       gazebo:='false'
+                      ft_sensor:='false'
                       with_sc:='false'
                       ros2_control:=false
@@ -44,4 +45,135 @@
       connected_to="${connected_to}"
     />
+    <xacro:if value="${ft_sensor and gazebo}">
+      <xacro:property name="connection" value="${arm_prefix_modified + arm_id + '_link8'}" />
+      <gazebo reference="${arm_prefix_modified} + joint7">
+        <sensor name="force_torque_sensor" type="force_torque">
+          <always_on>true</always_on>
+          <update_rate>50</update_rate>
+          <visualize>true</visualize>
+          <topic>wrist/force_torque</topic>
+          <force_torque>
+            <frame>sensor</frame>
+            <measure_direction>parent_to_child</measure_direction>
+          </force_torque>
+        </sensor>
+      </gazebo>
+      <!--plugin
+        filename="ignition-gazebo-forcetorque-system"
+        name="ignition::gazebo::systems::ForceTorque">
+      </plugin-->
+    </xacro:if>
+    <xacro:if value="${ft_sensor}">
+      <xacro:property name="connection" value="${arm_prefix_modified + arm_id + '_link8'}" />
+      <joint name="link8_ft_sensor_joint" type="fixed">
+        <parent link="${connection}"/>
+        <child link="${arm_prefix_modified + 'pre_ft_sensor_link'}"/>
+        <origin xyz="0 0 0.01" rpy="0 0 0"/>
+      </joint>
+      <joint name="pre_ft_sensor_joint" type="fixed">
+        <parent link="${arm_prefix_modified + 'pre_ft_sensor_link'}"/>
+        <child link="${arm_prefix_modified + 'nordbo_ft_sensor_link'}"/>
+        <origin xyz="0 0 0.021" rpy="0 0 0"/>
+      </joint>
+      <joint name="post_ft_sensor_joint" type="fixed">
+        <parent link="${arm_prefix_modified + 'nordbo_ft_sensor_link'}"/>
+        <child link="${arm_prefix_modified + 'post_ft_sensor_link'}"/>
+        <origin xyz="0 0 0.021" rpy="0 0 0"/>
+      </joint>
+      <joint name="gripper_coupling_joint" type="fixed">
+        <parent link="${arm_prefix_modified + 'post_ft_sensor_link'}"/>
+        <child link="${arm_prefix_modified + 'coupling_robotiq_link'}"/>
+        <origin xyz="0 0 0.01695" rpy="0 0 0"/>
+      </joint>
+      <joint name="tool0_joint" type="fixed">
+        <parent link="${arm_prefix_modified + 'coupling_robotiq_link'}"/>
+        <child link="${arm_prefix_modified + 'tool0'}"/>
+        <origin xyz="0 0 0.00695" rpy="0 0 0"/>
+      </joint>
+      <link name="${arm_prefix_modified + 'pre_ft_sensor_link'}">
+        <visual>
+          <geometry>
+            <cylinder radius="0.0375" length="0.02"/>
+          </geometry>
+          <material name="black">
+            <color rgba="0 0 0 1"/>
+          </material>
+        </visual>
+        <collision>
+          <geometry>
+            <cylinder radius="0.0375" length="0.02"/>
+          </geometry>
+        </collision>
+        <inertial>
+          <mass value="0.09"/>
+          <origin xyz="0 0 0" rpy="0 0 0"/>
+          <inertia ixx="3.46e-5" iyy="3.46e-5" izz="6.33e-5" ixy="0.0" ixz="0.0" iyz="0.0"/>
+        </inertial>
+      </link>
+      <link name="${arm_prefix_modified + 'nordbo_ft_sensor_link'}">
+        <visual>
+          <geometry>
+            <cylinder radius="0.025" length="0.022"/>
+          </geometry>
+          <material name="blue">
+            <color rgba="0 0.557 0.8 1"/>
+          </material>
+        </visual>
+        <collision>
+          <geometry>
+            <cylinder radius="0.025" length="0.022"/>
+          </geometry>
+        </collision>
+        <inertial>
+          <mass value="0.1"/>
+          <origin xyz="0 0 0" rpy="0 0 0"/>
+          <inertia ixx="1.97e-5" iyy="1.97e-5" izz="3.125e-5" ixy="0.0" ixz="0.0" iyz="0.0"/>
+        </inertial>
+      </link>
+      <link name="${arm_prefix_modified + 'post_ft_sensor_link'}">
+        <visual>
+          <geometry>
+            <cylinder radius="0.0375" length="0.02"/>
+          </geometry>
+          <material name="black">
+            <color rgba="0 0 0 1"/>
+          </material>
+        </visual>
+        <collision>
+          <geometry>
+            <cylinder radius="0.0375" length="0.02"/>
+          </geometry>
+        </collision>
+        <inertial>
+          <mass value="0.09"/>
+          <origin xyz="0 0 0" rpy="0 0 0"/>
+          <inertia ixx="3.46e-5" iyy="3.46e-5" izz="6.33e-5" ixy="0.0" ixz="0.0" iyz="0.0"/>
+        </inertial>
+      </link>
+      <link name="${arm_prefix_modified + 'coupling_robotiq_link'}">
+        <visual>
+          <geometry>
+            <!--cylinder radius="0.0375" length="0.0169"/-->
+            <cylinder radius="0.0375" length="0.0139"/>
+          </geometry>
+          <material name="black">
+            <color rgba="0 0 0 1"/>
+          </material>
+        </visual>
+        <collision>
+          <geometry>
+            <!--cylinder radius="0.0375" length="0.0169"/-->
+            <cylinder radius="0.0375" length="0.005"/>
+          </geometry>
+        </collision>
+        <inertial>
+          <mass value="0.0355"/> <!--DOUBLE CHECK-->
+          <origin xyz="0 0 0" rpy="0 0 0"/>
+          <inertia ixx="1.33e-5" iyy="1.33e-5" izz="2.5e-5" ixy="0.0" ixz="0.0" iyz="0.0"/>
+        </inertial>
+      </link>
+      <link name="${arm_prefix_modified + 'tool0'}">
+      </link>
+    </xacro:if>
     <xacro:if value="${hand and ee_id == 'franka_hand'}">
       <xacro:include filename="$(find franka_description)/end_effectors/common/franka_hand.xacro"/>
@@ -78,4 +210,7 @@
       <xacro:property name="ee_color" value="black" />
       <xacro:property name="connection" value="${arm_prefix_modified + arm_id + '_link8'}" />
+      <xacro:if value="${ft_sensor}">
+        <xacro:property name="connection" value="${arm_prefix_modified + 'tool0'}" />
+      </xacro:if>
       <xacro:robotiq_gripper name="RobotiqGripperHardwareInterface" prefix="${arm_prefix_modified}" parent="${connection}" use_fake_hardware="$(arg use_fake_hardware)" com_port="$(arg com_port)" sim_ignition="${gazebo}" robot="true">
         <origin xyz="0 0 0" rpy="0 0 0" />
