Commit message: developments

File: franka_robotiq/urdf/2f_85.ros2_control.xacro (robot description, xacro)
@@ -18,5 +18,5 @@
         gripper_max_force:=235.0
         gripper_closed_position:=0.7929">
-        <ros2_control name="${prefix + name}" type="system">
+        <ros2_control name="${prefix + name}TEST" type="system">
             <!-- Plugins -->
             <!--xacro:unless value="${robot and sim_ignition}"-->

File: franka_robotiq/urdf/fr3_robotiq.urdf.xacro (robot description, xacro)
@@ -15,4 +15,5 @@
   <!-- Should an end-effector be mounted at the flange?" -->
   <xacro:arg name="hand" default="true" />
+  <xacro:arg name="hand_control" default="true" />
   <!-- Which end-effector would be mounted at the flange?" -->
   <xacro:arg name="ee_id" default="robotiq" />
@@ -49,4 +50,5 @@
                       gazebo="$(arg gazebo)"
                       hand="$(arg hand)"
+                      hand_control="$(arg hand_control)"
                       ee_id="$(arg ee_id)"
                       with_sc="$(arg with_sc)"

File: franka_robotiq/urdf/franka_arm.ros2_control.xacro (robot description, xacro)
@@ -72,66 +72,4 @@
         <xacro:configure_joint joint_name="${arm_id}_finger_joint1" initial_position="0.0" />
       </xacro:if>
-      <!--xacro:if value="${gazebo and hand and ee_id == 'robotiq'}">
-            <joint name="${arm_prefix_modified}robotiq_85_left_knuckle_joint">
-                <command_interface name="position" />
-                <state_interface name="position">
-                    <param name="initial_value">${gripper_closed_position}</param>
-                </state_interface>
-                <state_interface name="velocity"/>
-            </joint>
-            <xacro:if value="${use_fake_hardware or gazebo}">
-                <joint name="${arm_prefix_modified}robotiq_85_right_knuckle_joint">
-                    <param name="mimic">${arm_prefix_modified}robotiq_85_left_knuckle_joint</param>
-                    <param name="multiplier">-1</param>
-                    <xacro:unless value="${gazebo}">
-                        <command_interface name="position"/>
-                        <state_interface name="position"/>
-                        <state_interface name="velocity"/>
-                    </xacro:unless>
-                </joint>
-                <joint name="${arm_prefix_modified}robotiq_85_left_inner_knuckle_joint">
-                    <param name="mimic">${arm_prefix_modified}robotiq_85_left_knuckle_joint</param>
-                    <param name="multiplier">1</param>
-                    <xacro:unless value="${gazebo}">
-                        <command_interface name="position"/>
-                        <state_interface name="position"/>
-                        <state_interface name="velocity"/>
-                    </xacro:unless>
-                </joint>
-                <joint name="${arm_prefix_modified}robotiq_85_right_inner_knuckle_joint">
-                    <param name="mimic">${arm_prefix_modified}robotiq_85_left_knuckle_joint</param>
-                    <param name="multiplier">-1</param>
-                    <xacro:unless value="${gazebo}">
-                        <command_interface name="position"/>
-                        <state_interface name="position"/>
-                        <state_interface name="velocity"/>
-                    </xacro:unless>
-                </joint>
-                <joint name="${arm_prefix_modified}robotiq_85_left_finger_tip_joint">
-                    <param name="mimic">${arm_prefix_modified}robotiq_85_left_knuckle_joint</param>
-                    <param name="multiplier">-1</param>
-                    <xacro:unless value="${gazebo}">
-                        <command_interface name="position"/>
-                        <state_interface name="position"/>
-                        <state_interface name="velocity"/>
-                    </xacro:unless>
-                </joint>
-                <joint name="${arm_prefix_modified}robotiq_85_right_finger_tip_joint">
-                    <param name="mimic">${arm_prefix_modified}robotiq_85_left_knuckle_joint</param>
-                    <param name="multiplier">1</param>
-                    <xacro:unless value="${gazebo}">
-                        <command_interface name="position"/>
-                        <state_interface name="position"/>
-                        <state_interface name="velocity"/>
-                    </xacro:unless>
-                </joint>
-            </xacro:if>
-            <xacro:unless value="${gazebo}">
-                <gpio name="reactivate_gripper">
-                    <command_interface name="reactivate_gripper_cmd" />
-                    <command_interface name="reactivate_gripper_response" />
-                </gpio>
-            </xacro:unless>
-      </xacro:if-->
     </ros2_control>
     <xacro:if value="${gazebo}">

File: franka_robotiq/urdf/franka_robotiq.xacro (robot description, xacro)
@@ -11,4 +11,5 @@
                       rpy:='0 0 0'
                       hand:='true'
+                      hand_control:='true'
                       ee_id:='franka_hand'
                       gazebo:='false'
@@ -89,5 +90,5 @@
         <parent link="${arm_prefix_modified + 'coupling_robotiq_link'}"/>
         <child link="${arm_prefix_modified + 'tool0'}"/>
-        <origin xyz="0 0 0.00695" rpy="0 0 0"/>
+        <origin xyz="0 0 0.00695" rpy="0 0 0.7854"/>
       </joint>
       <link name="${arm_prefix_modified + 'pre_ft_sensor_link'}">
@@ -213,7 +214,42 @@
         <xacro:property name="connection" value="${arm_prefix_modified + 'tool0'}" />
       </xacro:if>
-      <xacro:robotiq_gripper name="RobotiqGripperHardwareInterface" prefix="${arm_prefix_modified}" parent="${connection}" use_fake_hardware="$(arg use_fake_hardware)" com_port="$(arg com_port)" sim_ignition="${gazebo}" robot="true">
-        <origin xyz="0 0 0" rpy="0 0 0" />
-      </xacro:robotiq_gripper>
+      <xacro:if value="${hand_control}">
+        <xacro:robotiq_gripper name="RobotiqGripperHardwareInterface" prefix="${arm_prefix_modified}" parent="${connection}" use_fake_hardware="$(arg use_fake_hardware)" com_port="$(arg com_port)" sim_ignition="${gazebo}" robot="true">
+          <origin xyz="0 0 0" rpy="0 0 0" />
+        </xacro:robotiq_gripper>
+      </xacro:if>
+      <xacro:unless value="${hand_control}">
+        <joint name="gripper_collisions_joint" type="fixed">
+          <parent link="${arm_prefix_modified + 'tool0'}"/>
+          <child link="gripper_collisions"/>
+          <origin xyz="0 0 0.08005" rpy="0 0 0"/>
+        </joint>
+        <joint name="tcp_collisions_joint" type="fixed">
+          <parent link="gripper_collisions"/>
+          <child link="tcp"/>
+          <origin xyz="0 0 0.08005" rpy="0 0 0"/>
+        </joint>
+        <link name="gripper_collisions">
+          <visual>
+            <geometry>
+              <cylinder radius="0.0375" length="0.1601"/>
+            </geometry>
+            <material name="collision_color">
+              <color rgba="1 0 0 0"/>
+            </material>
+          </visual>
+          <collision>
+            <geometry>
+              <cylinder radius="0.0375" length="0.1601"/>
+            </geometry>
+          </collision>
+          <inertial>
+            <mass value="0.8895"/>
+            <origin xyz="0 0 0" rpy="0 0 0"/>
+            <inertia ixx="0.00418" iyy="0.00508" izz="0.00125" ixy="0.0" ixz="0.0" iyz="0.0"/>
+          </inertial>
+        </link>
+        <link name="tcp"/>
+      </xacro:unless>
     </xacro:if>
     <xacro:if value="${hand and ee_id != 'none' and ee_id != 'franka_hand' and ee_id != 'robotiq'}">

File: franka_robotiq_moveit_config/config/fr3_ft_sensor.srdf.xacro (robot description, xacro)
@@ -189,8 +189,9 @@
     <disable_collisions link1="robotiq_85_right_finger_tip_link" link2="robotiq_85_right_knuckle_link" reason="Never"/>
     <disable_collisions link1="robotiq_85_right_inner_knuckle_link" link2="robotiq_85_right_knuckle_link" reason="Never"/>
-    <disable_collisions link1="fr3_link8" link2="pre_ft_sensor_link" reason="Adjacent"/>
+    <disable_collisions link1="fr3_link7" link2="pre_ft_sensor_link" reason="Never"/>
+    <!--disable_collisions link1="fr3_link8" link2="pre_ft_sensor_link" reason="Adjacent"/-->
     <disable_collisions link1="pre_ft_sensor_link" link2="nordbo_ft_sensor_link" reason="Adjacent"/>
     <disable_collisions link1="nordbo_ft_sensor_link" link2="post_ft_sensor_link" reason="Adjacent"/>
     <disable_collisions link1="post_ft_sensor_link" link2="coupling_robotiq_link" reason="Adjacent"/>
-    <disable_collisions link1="coupling_robotiq_link" link2="robotiq_85_base_link" reason="Adjacent"/>
+    <disable_collisions link1="coupling_robotiq_link" link2="robotiq_85_base_link" reason="Never"/>
 </robot>
