Commit message: controllers force sensors and aruco tracker

File: franka_robotiq/urdf/fr3_ft_sensor.srdf.xacro (robot description, xacro)
@@ -60,4 +60,31 @@
         <joint name="fr3_joint7" value="1.283"/>
     </group_state>
+    <group_state name="ready" group="fr3_arm">
+        <joint name="fr3_joint1" value="0"/>
+        <joint name="fr3_joint2" value="-0.785"/>
+        <joint name="fr3_joint3" value="0"/>
+        <joint name="fr3_joint4" value="-2.356"/>
+        <joint name="fr3_joint5" value="0"/>
+        <joint name="fr3_joint6" value="1.571"/>
+        <joint name="fr3_joint7" value="0.785"/>
+    </group_state>
+    <group_state name="ready_kaleel" group="fr3_arm">
+        <joint name="fr3_joint1" value="0.0019290960160640493"/>
+        <joint name="fr3_joint2" value="-0.07429991145403866"/>
+        <joint name="fr3_joint3" value="0.0009094689629045991"/>
+        <joint name="fr3_joint4" value="-2.7644865457325847"/>
+        <joint name="fr3_joint5" value="-0.0015472140117172208"/>
+        <joint name="fr3_joint6" value="2.686926798618501"/>
+        <joint name="fr3_joint7" value="0.7922321460407836"/>
+    </group_state>
+    <group_state name="ready_ses_rod" group="fr3_arm">
+        <joint name="fr3_joint1" value="0.36431833142346814"/>
+        <joint name="fr3_joint2" value="-0.19478917595231374"/>
+        <joint name="fr3_joint3" value="-0.0069491493639888486"/>
+        <joint name="fr3_joint4" value="-2.1238954117435624"/>
+        <joint name="fr3_joint5" value="-0.002320934374129336"/>
+        <joint name="fr3_joint6" value="1.912285393484237"/>
+        <joint name="fr3_joint7" value="1.1365761522738094"/>
+    </group_state>
     <!--END EFFECTOR: Purpose: Represent information about an end effector.-->
     <!--PASSIVE JOINT: Purpose: this element is used to mark joints that are not actuated-->

File: franka_robotiq/urdf/fr3_robotiq.urdf.xacro (robot description, xacro)
@@ -14,5 +14,5 @@
   <xacro:arg name="arm_prefix" default=""/>
   <!-- Should an end-effector be mounted at the flange?" -->
-  <xacro:arg name="hand" default="true" />
+  <xacro:arg name="hand" default="false" />
   <xacro:arg name="hand_control" default="true" />
   <!-- Which end-effector would be mounted at the flange?" -->

File: franka_robotiq/urdf/franka_arm.ros2_control.xacro (robot description, xacro)
@@ -72,4 +72,28 @@
         <xacro:configure_joint joint_name="${arm_id}_finger_joint1" initial_position="0.0" />
       </xacro:if>
+      <xacro:macro name="general_purpose_io" params="prefix command_interface index">
+        <gpio name="${prefix}">
+          <command_interface name="${command_interface}"/>
+          <param name="index">${index}</param>
+        </gpio>
+      </xacro:macro>
+      <!-- Cartesian velocity interfaces -->
+      <xacro:general_purpose_io prefix="vx" command_interface="cartesian_velocity" index="0"/>
+      <xacro:general_purpose_io prefix="vy" command_interface="cartesian_velocity" index="1"/>
+      <xacro:general_purpose_io prefix="vz" command_interface="cartesian_velocity" index="2"/>
+      <xacro:general_purpose_io prefix="wx" command_interface="cartesian_velocity" index="3"/>
+      <xacro:general_purpose_io prefix="wy" command_interface="cartesian_velocity" index="4"/>
+      <xacro:general_purpose_io prefix="wz" command_interface="cartesian_velocity" index="5"/>
+      <!-- Cartesian pose interfaces, in total 16 interfaces -->
+      <xacro:macro name="loop" params="i">
+        <xacro:unless value="${i == 16}">
+          <xacro:general_purpose_io prefix="${i}" command_interface="cartesian_pose_command" index="${i}"/>
+          <xacro:loop i="${i+1}"/>
+        </xacro:unless>
+      </xacro:macro>
+      <xacro:loop i="0"/>
+      <!-- Elbow command interfaces -->
+      <xacro:general_purpose_io prefix="joint_3_position" command_interface="elbow_command" index="0"/>
+      <xacro:general_purpose_io prefix="joint_4_sign" command_interface="elbow_command" index="1"/>
     </ros2_control>
     <xacro:if value="${gazebo}">

File: franka_robotiq/urdf/franka_robotiq.xacro (robot description, xacro)
@@ -70,5 +70,5 @@
         <parent link="${connection}"/>
         <child link="${arm_prefix_modified + 'pre_ft_sensor_link'}"/>
-        <origin xyz="0 0 0.01" rpy="0 0 0"/>
+        <origin xyz="0 0 0.01" rpy="0 0 0.7854"/>
       </joint>
       <joint name="pre_ft_sensor_joint" type="fixed">
@@ -90,5 +90,5 @@
         <parent link="${arm_prefix_modified + 'coupling_robotiq_link'}"/>
         <child link="${arm_prefix_modified + 'tool0'}"/>
-        <origin xyz="0 0 0.00695" rpy="0 0 0.7854"/>
+        <origin xyz="0 0 0.00695" rpy="0 0 0"/>
       </joint>
       <link name="${arm_prefix_modified + 'pre_ft_sensor_link'}">

Commit message: exp_chain

File: franka_robotiq/urdf/fr3_ft_sensor.srdf.xacro (robot description, xacro)
@@ -87,4 +87,13 @@
         <joint name="fr3_joint7" value="1.1365761522738094"/>
     </group_state>
+    <group_state name="ready_ses_chain" group="fr3_arm">
+        <joint name="fr3_joint1" value="0.46423243854334867"/>
+        <joint name="fr3_joint2" value="-0.8532201615854992"/>
+        <joint name="fr3_joint3" value="0.1139657812019727"/>
+        <joint name="fr3_joint4" value="-2.626267858279923"/>
+        <joint name="fr3_joint5" value="0.08784949911892842"/>
+        <joint name="fr3_joint6" value="1.7589591080624436"/>
+        <joint name="fr3_joint7" value="1.2930822900254497"/>
+    </group_state>
     <!--END EFFECTOR: Purpose: Represent information about an end effector.-->
     <!--PASSIVE JOINT: Purpose: this element is used to mark joints that are not actuated-->

Commit message: real_experiments

File: franka_robotiq/urdf/fr3_ft_sensor.srdf.xacro (robot description, xacro)
@@ -96,4 +96,22 @@
         <joint name="fr3_joint7" value="1.2930822900254497"/>
     </group_state>
+    <group_state name="ready_ses_ring" group="fr3_arm">
+        <joint name="fr3_joint1" value="0.3887571125646938"/>
+        <joint name="fr3_joint2" value="-0.4167294414542532"/>
+        <joint name="fr3_joint3" value="0.02992998976402808"/>
+        <joint name="fr3_joint4" value="-2.3348725998664532"/>
+        <joint name="fr3_joint5" value="0.013494065988005836"/>
+        <joint name="fr3_joint6" value="1.8983932197171471"/>
+        <joint name="fr3_joint7" value="1.190480320908703"/>
+    </group_state>
+    <group_state name="ready_ses_branch" group="fr3_arm">
+        <joint name="fr3_joint1" value="0.4391810214519501"/>
+        <joint name="fr3_joint2" value="-0.6843689606200062"/>
+        <joint name="fr3_joint3" value="0.09142039648174596"/>
+        <joint name="fr3_joint4" value="-2.5324462799851704"/>
+        <joint name="fr3_joint5" value="0.06089145710157039"/>
+        <joint name="fr3_joint6" value="1.8311098529480945"/>
+        <joint name="fr3_joint7" value="1.2720793133431665"/>
+    </group_state>
     <!--END EFFECTOR: Purpose: Represent information about an end effector.-->
     <!--PASSIVE JOINT: Purpose: this element is used to mark joints that are not actuated-->

Commit message: visibility_disturbances_exp

File: franka_robotiq/urdf/fr3_ft_sensor.srdf.xacro (robot description, xacro)
@@ -114,4 +114,22 @@
         <joint name="fr3_joint7" value="1.2720793133431665"/>
     </group_state>
+    <group_state name="ready_ses_branch_low" group="fr3_arm">
+        <joint name="fr3_joint1" value="0.36538194441109245"/>
+        <joint name="fr3_joint2" value="-0.2037238491011323"/>
+        <joint name="fr3_joint3" value="0.036152998080117106"/>
+        <joint name="fr3_joint4" value="-2.4648117770046043"/>
+        <joint name="fr3_joint5" value="-0.010086970275305612"/>
+        <joint name="fr3_joint6" value="2.2132315249277674"/>
+        <joint name="fr3_joint7" value="1.132772110688066"/>
+    </group_state>
+    <group_state name="ready_ses_visibility" group="fr3_arm">
+        <joint name="fr3_joint1" value="0.2540970409259686"/>
+        <joint name="fr3_joint2" value="-0.6775709692804806"/>
+        <joint name="fr3_joint3" value="-0.2965978402626135"/>
+        <joint name="fr3_joint4" value="-2.506488201583876"/>
+        <joint name="fr3_joint5" value="-0.21344199732591798"/>
+        <joint name="fr3_joint6" value="1.8289728196853776"/>
+        <joint name="fr3_joint7" value="0.8405917357170101"/>
+    </group_state>
     <!--END EFFECTOR: Purpose: Represent information about an end effector.-->
     <!--PASSIVE JOINT: Purpose: this element is used to mark joints that are not actuated-->
