Commit message: visibility_disturbances_exp 2

File: franka_robotiq/urdf/fr3_ft_sensor.srdf.xacro (robot description, xacro)
@@ -1,160 +1,127 @@
-<?xml version="1.0" encoding="UTF-8"?>
-<!--This does not replace URDF, and is not an extension of URDF.
-    This is a format for representing semantic information about the robot structure.
-    A URDF file must exist for this robot as well, where the joints and the links that are referenced are defined
--->
-<robot xmlns:xacro="http://www.ros.org/wiki/xacro" name="fr3">
-    <!--GROUPS: Representation of a set of joints and links. This can be useful for specifying DOF to plan for, defining arms, end effectors, etc-->
-    <!--LINKS: When a link is specified, the parent joint of that link (if it exists) is automatically included-->
-    <!--JOINTS: When a joint is specified, the child link of that joint (which will always exist) is automatically included-->
-    <!--CHAINS: When a chain is specified, all the links along the chain (including endpoints) are included in the group. Additionally, all the joints that are parents to included links are also included. This means that joints along the chain and the parent joint of the base link are included in the group-->
-    <!--SUBGROUPS: Groups can also be formed by referencing to already defined group names-->
-    <!--group name="franka_arm">
-        <link name="base"/>
-        <link name="fr3_link0"/>
-        <link name="fr3_link1"/>
-        <link name="fr3_link2"/>
-        <link name="fr3_link3"/>
-        <link name="fr3_link4"/>
-        <link name="fr3_link5"/>
-        <link name="fr3_link6"/>
-        <link name="fr3_link7"/>
-        <link name="fr3_link8"/>
-        <joint name="fr3_joint1"/>
-        <joint name="fr3_joint7"/>
-        <joint name="fr3_joint6"/>
-        <joint name="fr3_joint5"/>
-        <joint name="fr3_joint4"/>
-        <joint name="fr3_joint3"/>
-        <joint name="fr3_joint2"/>
-    </group-->
+<?xml version='1.0' encoding='utf-8'?>
+<robot name="fr3">
     <group name="fr3_arm">
-        <chain base_link="fr3_link0" tip_link="tool0"/>
+        <chain base_link="fr3_link0" tip_link="tool0" />
     </group>
-    <!--GROUP STATES: Purpose: Define a named state for a particular group, in terms of joint values. This is useful to define states like 'folded arms'-->
     <group_state name="home" group="fr3_arm">
-        <joint name="fr3_joint1" value="0"/>
-        <joint name="fr3_joint2" value="0"/>
-        <joint name="fr3_joint3" value="0"/>
-        <joint name="fr3_joint4" value="-1.59695"/>
-        <joint name="fr3_joint5" value="0"/>
-        <joint name="fr3_joint6" value="2.5307"/>
-        <joint name="fr3_joint7" value="0"/>
+        <joint name="fr3_joint1" value="0" />
+        <joint name="fr3_joint2" value="0" />
+        <joint name="fr3_joint3" value="0" />
+        <joint name="fr3_joint4" value="-1.59695" />
+        <joint name="fr3_joint5" value="0" />
+        <joint name="fr3_joint6" value="2.5307" />
+        <joint name="fr3_joint7" value="0" />
     </group_state>
     <group_state name="up" group="fr3_arm">
-        <joint name="fr3_joint1" value="0"/>
-        <joint name="fr3_joint2" value="0"/>
-        <joint name="fr3_joint3" value="0"/>
-        <joint name="fr3_joint4" value="-0.2"/>
-        <joint name="fr3_joint5" value="0"/>
-        <joint name="fr3_joint6" value="3.14"/>
-        <joint name="fr3_joint7" value="0"/>
+        <joint name="fr3_joint1" value="0" />
+        <joint name="fr3_joint2" value="0" />
+        <joint name="fr3_joint3" value="0" />
+        <joint name="fr3_joint4" value="-0.2" />
+        <joint name="fr3_joint5" value="0" />
+        <joint name="fr3_joint6" value="3.14" />
+        <joint name="fr3_joint7" value="0" />
     </group_state>
     <group_state name="random" group="fr3_arm">
-        <joint name="fr3_joint1" value="1.5916"/>
-        <joint name="fr3_joint2" value="0.5617"/>
-        <joint name="fr3_joint3" value="0"/>
-        <joint name="fr3_joint4" value="-1.2856"/>
-        <joint name="fr3_joint5" value="1.1319"/>
-        <joint name="fr3_joint6" value="2.5636"/>
-        <joint name="fr3_joint7" value="1.283"/>
+        <joint name="fr3_joint1" value="1.5916" />
+        <joint name="fr3_joint2" value="0.5617" />
+        <joint name="fr3_joint3" value="0" />
+        <joint name="fr3_joint4" value="-1.2856" />
+        <joint name="fr3_joint5" value="1.1319" />
+        <joint name="fr3_joint6" value="2.5636" />
+        <joint name="fr3_joint7" value="1.283" />
     </group_state>
     <group_state name="ready" group="fr3_arm">
-        <joint name="fr3_joint1" value="0"/>
-        <joint name="fr3_joint2" value="-0.785"/>
-        <joint name="fr3_joint3" value="0"/>
-        <joint name="fr3_joint4" value="-2.356"/>
-        <joint name="fr3_joint5" value="0"/>
-        <joint name="fr3_joint6" value="1.571"/>
-        <joint name="fr3_joint7" value="0.785"/>
+        <joint name="fr3_joint1" value="0" />
+        <joint name="fr3_joint2" value="-0.785" />
+        <joint name="fr3_joint3" value="0" />
+        <joint name="fr3_joint4" value="-2.356" />
+        <joint name="fr3_joint5" value="0" />
+        <joint name="fr3_joint6" value="1.571" />
+        <joint name="fr3_joint7" value="0.785" />
     </group_state>
     <group_state name="ready_kaleel" group="fr3_arm">
-        <joint name="fr3_joint1" value="0.0019290960160640493"/>
-        <joint name="fr3_joint2" value="-0.07429991145403866"/>
-        <joint name="fr3_joint3" value="0.0009094689629045991"/>
-        <joint name="fr3_joint4" value="-2.7644865457325847"/>
-        <joint name="fr3_joint5" value="-0.0015472140117172208"/>
-        <joint name="fr3_joint6" value="2.686926798618501"/>
-        <joint name="fr3_joint7" value="0.7922321460407836"/>
+        <joint name="fr3_joint1" value="0.0019290960160640493" />
+        <joint name="fr3_joint2" value="-0.07429991145403866" />
+        <joint name="fr3_joint3" value="0.0009094689629045991" />
+        <joint name="fr3_joint4" value="-2.7644865457325847" />
+        <joint name="fr3_joint5" value="-0.0015472140117172208" />
+        <joint name="fr3_joint6" value="2.686926798618501" />
+        <joint name="fr3_joint7" value="0.7922321460407836" />
     </group_state>
     <group_state name="ready_ses_rod" group="fr3_arm">
-        <joint name="fr3_joint1" value="0.36431833142346814"/>
-        <joint name="fr3_joint2" value="-0.19478917595231374"/>
-        <joint name="fr3_joint3" value="-0.0069491493639888486"/>
-        <joint name="fr3_joint4" value="-2.1238954117435624"/>
-        <joint name="fr3_joint5" value="-0.002320934374129336"/>
-        <joint name="fr3_joint6" value="1.912285393484237"/>
-        <joint name="fr3_joint7" value="1.1365761522738094"/>
+        <joint name="fr3_joint1" value="0.36431833142346814" />
+        <joint name="fr3_joint2" value="-0.19478917595231374" />
+        <joint name="fr3_joint3" value="-0.0069491493639888486" />
+        <joint name="fr3_joint4" value="-2.1238954117435624" />
+        <joint name="fr3_joint5" value="-0.002320934374129336" />
+        <joint name="fr3_joint6" value="1.912285393484237" />
+        <joint name="fr3_joint7" value="1.1365761522738094" />
     </group_state>
     <group_state name="ready_ses_chain" group="fr3_arm">
-        <joint name="fr3_joint1" value="0.46423243854334867"/>
-        <joint name="fr3_joint2" value="-0.8532201615854992"/>
-        <joint name="fr3_joint3" value="0.1139657812019727"/>
-        <joint name="fr3_joint4" value="-2.626267858279923"/>
-        <joint name="fr3_joint5" value="0.08784949911892842"/>
-        <joint name="fr3_joint6" value="1.7589591080624436"/>
-        <joint name="fr3_joint7" value="1.2930822900254497"/>
+        <joint name="fr3_joint1" value="0.46423243854334867" />
+        <joint name="fr3_joint2" value="-0.8532201615854992" />
+        <joint name="fr3_joint3" value="0.1139657812019727" />
+        <joint name="fr3_joint4" value="-2.626267858279923" />
+        <joint name="fr3_joint5" value="0.08784949911892842" />
+        <joint name="fr3_joint6" value="1.7589591080624436" />
+        <joint name="fr3_joint7" value="1.2930822900254497" />
     </group_state>
     <group_state name="ready_ses_ring" group="fr3_arm">
-        <joint name="fr3_joint1" value="0.3887571125646938"/>
-        <joint name="fr3_joint2" value="-0.4167294414542532"/>
-        <joint name="fr3_joint3" value="0.02992998976402808"/>
-        <joint name="fr3_joint4" value="-2.3348725998664532"/>
-        <joint name="fr3_joint5" value="0.013494065988005836"/>
-        <joint name="fr3_joint6" value="1.8983932197171471"/>
-        <joint name="fr3_joint7" value="1.190480320908703"/>
+        <joint name="fr3_joint1" value="0.3887571125646938" />
+        <joint name="fr3_joint2" value="-0.4167294414542532" />
+        <joint name="fr3_joint3" value="0.02992998976402808" />
+        <joint name="fr3_joint4" value="-2.3348725998664532" />
+        <joint name="fr3_joint5" value="0.013494065988005836" />
+        <joint name="fr3_joint6" value="1.8983932197171471" />
+        <joint name="fr3_joint7" value="1.190480320908703" />
     </group_state>
     <group_state name="ready_ses_branch" group="fr3_arm">
-        <joint name="fr3_joint1" value="0.4391810214519501"/>
-        <joint name="fr3_joint2" value="-0.6843689606200062"/>
-        <joint name="fr3_joint3" value="0.09142039648174596"/>
-        <joint name="fr3_joint4" value="-2.5324462799851704"/>
-        <joint name="fr3_joint5" value="0.06089145710157039"/>
-        <joint name="fr3_joint6" value="1.8311098529480945"/>
-        <joint name="fr3_joint7" value="1.2720793133431665"/>
+        <joint name="fr3_joint1" value="0.4391810214519501" />
+        <joint name="fr3_joint2" value="-0.6843689606200062" />
+        <joint name="fr3_joint3" value="0.09142039648174596" />
+        <joint name="fr3_joint4" value="-2.5324462799851704" />
+        <joint name="fr3_joint5" value="0.06089145710157039" />
+        <joint name="fr3_joint6" value="1.8311098529480945" />
+        <joint name="fr3_joint7" value="1.2720793133431665" />
     </group_state>
     <group_state name="ready_ses_branch_low" group="fr3_arm">
-        <joint name="fr3_joint1" value="0.36538194441109245"/>
-        <joint name="fr3_joint2" value="-0.2037238491011323"/>
-        <joint name="fr3_joint3" value="0.036152998080117106"/>
-        <joint name="fr3_joint4" value="-2.4648117770046043"/>
-        <joint name="fr3_joint5" value="-0.010086970275305612"/>
-        <joint name="fr3_joint6" value="2.2132315249277674"/>
-        <joint name="fr3_joint7" value="1.132772110688066"/>
+        <joint name="fr3_joint1" value="0.36538194441109245" />
+        <joint name="fr3_joint2" value="-0.2037238491011323" />
+        <joint name="fr3_joint3" value="0.036152998080117106" />
+        <joint name="fr3_joint4" value="-2.4648117770046043" />
+        <joint name="fr3_joint5" value="-0.010086970275305612" />
+        <joint name="fr3_joint6" value="2.2132315249277674" />
+        <joint name="fr3_joint7" value="1.132772110688066" />
     </group_state>
     <group_state name="ready_ses_visibility" group="fr3_arm">
-        <joint name="fr3_joint1" value="0.2540970409259686"/>
-        <joint name="fr3_joint2" value="-0.6775709692804806"/>
-        <joint name="fr3_joint3" value="-0.2965978402626135"/>
-        <joint name="fr3_joint4" value="-2.506488201583876"/>
-        <joint name="fr3_joint5" value="-0.21344199732591798"/>
-        <joint name="fr3_joint6" value="1.8289728196853776"/>
-        <joint name="fr3_joint7" value="0.8405917357170101"/>
+        <joint name="fr3_joint1" value="0.2540970409259686" />
+        <joint name="fr3_joint2" value="-0.6775709692804806" />
+        <joint name="fr3_joint3" value="-0.2965978402626135" />
+        <joint name="fr3_joint4" value="-2.506488201583876" />
+        <joint name="fr3_joint5" value="-0.21344199732591798" />
+        <joint name="fr3_joint6" value="1.8289728196853776" />
+        <joint name="fr3_joint7" value="0.8405917357170101" />
     </group_state>
-    <!--END EFFECTOR: Purpose: Represent information about an end effector.-->
-    <!--PASSIVE JOINT: Purpose: this element is used to mark joints that are not actuated-->
-    <!--DISABLE COLLISIONS: By default it is assumed that any link of the robot could potentially come into collision with any other link in the robot. This tag disables collision checking between a specified pair of links. -->
-    <disable_collisions link1="fr3_link0" link2="fr3_link1" reason="Adjacent"/>
-    <disable_collisions link1="fr3_link0" link2="fr3_link2" reason="Never"/>
-    <disable_collisions link1="fr3_link0" link2="fr3_link3" reason="Never"/>
-    <disable_collisions link1="fr3_link0" link2="fr3_link4" reason="Never"/>
-    <disable_collisions link1="fr3_link1" link2="fr3_link2" reason="Adjacent"/>
-    <disable_collisions link1="fr3_link1" link2="fr3_link3" reason="Never"/>
-    <disable_collisions link1="fr3_link1" link2="fr3_link4" reason="Never"/>
-    <disable_collisions link1="fr3_link2" link2="fr3_link3" reason="Adjacent"/>
-    <disable_collisions link1="fr3_link2" link2="fr3_link4" reason="Never"/>
-    <disable_collisions link1="fr3_link3" link2="fr3_link4" reason="Adjacent"/>
-    <disable_collisions link1="fr3_link3" link2="fr3_link5" reason="Never"/>
-    <disable_collisions link1="fr3_link3" link2="fr3_link6" reason="Never"/>
-    <disable_collisions link1="fr3_link3" link2="fr3_link7" reason="Never"/>
-    <disable_collisions link1="fr3_link4" link2="fr3_link5" reason="Adjacent"/>
-    <disable_collisions link1="fr3_link4" link2="fr3_link6" reason="Never"/>
-    <disable_collisions link1="fr3_link4" link2="fr3_link7" reason="Never"/>
-    <disable_collisions link1="fr3_link5" link2="fr3_link6" reason="Adjacent"/>
-    <disable_collisions link1="fr3_link6" link2="fr3_link7" reason="Adjacent"/>
-    <disable_collisions link1="fr3_link7" link2="pre_ft_sensor_link" reason="Never"/>
-    <!--disable_collisions link1="fr3_link8" link2="pre_ft_sensor_link" reason="Adjacent"/-->
-    <disable_collisions link1="pre_ft_sensor_link" link2="nordbo_ft_sensor_link" reason="Adjacent"/>
-    <disable_collisions link1="nordbo_ft_sensor_link" link2="post_ft_sensor_link" reason="Adjacent"/>
-    <disable_collisions link1="post_ft_sensor_link" link2="coupling_robotiq_link" reason="Adjacent"/>
+    <disable_collisions link1="fr3_link0" link2="fr3_link1" reason="Adjacent" />
+    <disable_collisions link1="fr3_link0" link2="fr3_link2" reason="Never" />
+    <disable_collisions link1="fr3_link0" link2="fr3_link3" reason="Never" />
+    <disable_collisions link1="fr3_link0" link2="fr3_link4" reason="Never" />
+    <disable_collisions link1="fr3_link1" link2="fr3_link2" reason="Adjacent" />
+    <disable_collisions link1="fr3_link1" link2="fr3_link3" reason="Never" />
+    <disable_collisions link1="fr3_link1" link2="fr3_link4" reason="Never" />
+    <disable_collisions link1="fr3_link2" link2="fr3_link3" reason="Adjacent" />
+    <disable_collisions link1="fr3_link2" link2="fr3_link4" reason="Never" />
+    <disable_collisions link1="fr3_link3" link2="fr3_link4" reason="Adjacent" />
+    <disable_collisions link1="fr3_link3" link2="fr3_link5" reason="Never" />
+    <disable_collisions link1="fr3_link3" link2="fr3_link6" reason="Never" />
+    <disable_collisions link1="fr3_link3" link2="fr3_link7" reason="Never" />
+    <disable_collisions link1="fr3_link4" link2="fr3_link5" reason="Adjacent" />
+    <disable_collisions link1="fr3_link4" link2="fr3_link6" reason="Never" />
+    <disable_collisions link1="fr3_link4" link2="fr3_link7" reason="Never" />
+    <disable_collisions link1="fr3_link5" link2="fr3_link6" reason="Adjacent" />
+    <disable_collisions link1="fr3_link6" link2="fr3_link7" reason="Adjacent" />
+    <disable_collisions link1="fr3_link7" link2="pre_ft_sensor_link" reason="Never" />
+    <disable_collisions link1="pre_ft_sensor_link" link2="nordbo_ft_sensor_link" reason="Adjacent" />
+    <disable_collisions link1="nordbo_ft_sensor_link" link2="post_ft_sensor_link" reason="Adjacent" />
+    <disable_collisions link1="post_ft_sensor_link" link2="coupling_robotiq_link" reason="Adjacent" />
 </robot>
